File: eagle-design/schematics.sch (EAGLE design)
At the start: 45 parts, among them IC1 7805T, J1 DCJ0202, K1 SRD-05VDC-SL-C, Q1 16Hz, T1 BC547, U1 ATMEGA328P-AU

Commit message: completed design
Parts:
- removed S1: (no value), switch-omron:10-XX
- added R21, R22: 10KΩ, resistor:R-US_R0805
- added X1: (no value), con-wago-500:W237-102
- LED_GREEN, LED_RED: device led:LED3MM -> led:LEDCHIPLED_0805
- R19: value 10K -> 10KΩ
- R7, R8: value 100Ω -> 220Ω
Connections:
- net 5V: now also R21.1, R22.1, X1-1.KL; no longer S1.P, S1.P1
- net GND: now also X1-2.KL; no longer S1.S, S1.S1
- net NC: now also X2-3.KL; no longer X2-1.KL
- net NO: now also X2-1.KL; no longer X2-3.KL
- net RX: now also U1.PD0
- net SCL: now also R22.2
- net SDA: now also R21.2
- net TX: now also U1.PD1
Other:
- note added: "SDA / SCL Connections"
- moved on the sheet: R18, U1
