File: eagle-design/schematics.brd (EAGLE design)
At the start: 139.7 x 67 mm, 47 parts, among them IC1 7805T, J1 DCJ0202, K1 SRD-05VDC-SL-C, Q1 16Hz, T1 BC547, U1 ATMEGA328P-AU

Commit message: Added missing connection
Routing:
- net 5V: track 330.2 -> 332.9 mm
Changed lines of the file:
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@@
 </layers>
 <board>
-<fusionsync huburn="a.cGVyc29uYWw6dWUyYTI1NDFm" projecturn="a.cGVyc29uYWw6dWUyYTI1NDFmIzIwMjAxMDA2MzM5ODc2MDgx" f3durn="urn:adsk.wipprod:dm.lineage:nrWloDwkQKefvX74mOgsZg" pcbguid="" lastpulledtime="" lastsyncedchangeguid="" latestrevisionid="1184bd50-7014-48fc-b872-ea82cf77e3a2" lastsyncedrevisionid="1184bd50-7014-48fc-b872-ea82cf77e3a2" lastboardhashguid="5352318f-7c8c-681a-3485-1142d5fd0d02" lastpushedtime="2021-08-28T05:39:19Z" linktopcb3d="true"/>
+<fusionsync huburn="a.cGVyc29uYWw6dWUyYTI1NDFm" projecturn="a.cGVyc29uYWw6dWUyYTI1NDFmIzIwMjAxMDA2MzM5ODc2MDgx" f3durn="urn:adsk.wipprod:dm.lineage:nrWloDwkQKefvX74mOgsZg" pcbguid="" lastpulledtime="" lastsyncedchangeguid="" latestrevisionid="cc03d767-f2ed-4469-88e5-19889d96c1c8" lastsyncedrevisionid="cc03d767-f2ed-4469-88e5-19889d96c1c8" lastboardhashguid="50b3749a-a130-4758-be0e-5e50d5d91a76" lastpushedtime="2021-08-28T16:38:54Z" linktopcb3d="true"/>
 <plain>
 <wire x1="0" y1="98.679" x2="0" y2="33.909" width="0" layer="20"/>
@@
 <wire x1="78.74" y1="35.6108" x2="78.74" y2="38.1" width="0.6096" layer="16"/>
 <wire x1="96.5708" y1="34.3408" x2="80.01" y2="34.3408" width="0.6096" layer="16"/>
-<wire x1="52.56" y1="45.32" x2="67.71" y2="45.32" width="0.6096" layer="1"/>
+<wire x1="52.56" y1="45.32" x2="60.217" y2="45.32" width="0.6096" layer="1"/>
 <via x="68.58" y="44.45" extent="1-16" drill="0.35"/>
+<wire x1="60.5028" y1="45.32" x2="67.71" y2="45.32" width="0.6096" layer="1"/>
 <wire x1="67.71" y1="45.32" x2="68.58" y2="44.45" width="0.6096" layer="1"/>
 <wire x1="71.12" y1="41.91" x2="68.58" y2="44.45" width="0.6096" layer="16"/>
@@
 <vertex x="138.303" y="99.822"/>
 </polygon>
+<wire x1="58.293" y1="47.244" x2="60.217" y2="45.32" width="0.6096" layer="1"/>
+<wire x1="60.217" y1="45.32" x2="60.5028" y2="45.32" width="0.6096" layer="1"/>
 </signal>
 <signal name="N$1">
@@
 <mfgpreviewcolor name="substratecolor" color="0xFF786E46"/>
 </mfgpreviewcolors>
+<errors>
+</errors>
 </board>
 </drawing>
